File: pcb/grapefruit-board.sch (EAGLE design)
At the start: 154 parts, among them IC1 L70, IC10 TS520525, IC2 STC3100, IC3 TPS61200, IC4 LM3671MF, IC5 MCP73837MF, IC6 LM2840/1/2, IC7 STM32F411XC, IC8 S25FL064K, IC9 TLV320AIC3100, M1 ELECTRET_MICROPHON-WM-62PC/62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, Q1 BSS84, Q2 BSS84, Q3 BSS84, Q4 BSS84, X1 BU-SMA-V, X2 BU-SMA-V, X3 BU-SMA-V, X4 USB-MICROB, X5 USB-MICROB, Y1 32768Hz

Commit message: Resolve the remaining unconnected parts
Parts:
- removed LED6, LED7: (no value), led:LEDCHIP-LED0603
- removed R26, R27: 1K, rcl:R-EU_R0603
- added C59, C63, C64, C65: 100nF, rcl:C-EUC0603
- added C60, C61, C62: 1uF, rcl:C-EUC0603
- added R34: 100K, rcl:R-EU_R0603
- added R35: 47K, rcl:R-EU_R0603
- added R36: 27K, rcl:R-EU_R0603
- added R37: 10K, rcl:R-EU_R0603
Connections:
- removed net CHG_FULL: IC5.STAT2
- removed net CHG_PG: IC5.PG
- removed net CODEC_RESET: IC9.RESET
- removed net N$33: LED6.A, R26.1
- removed net N$34: LED7.A, R27.1
- removed net R12_MISO: RFM22B_23B_26W.SDO, RFM22B_23B_26W1.SDO, RFM69W_69HW.MISO, RFM69W_69HW1.MISO
- removed net R12_MOSI: RFM22B_23B_26W.SDI, RFM22B_23B_26W1.SDI, RFM69W_69HW.MOSI, RFM69W_69HW1.MOSI
- removed net R12_SCK: RFM22B_23B_26W.SCK, RFM22B_23B_26W1.SCK, RFM69W_69HW.SCK, RFM69W_69HW1.SCK
- removed net R1_DIO1: RFM22B_23B_26W.GPIO1, RFM69W_69HW.DIO1
- removed net R1_DIO3: RFM22B_23B_26W.GPIO3, RFM69W_69HW.DIO3
- removed net R1_DIO4: RFM22B_23B_26W.NIRQ, RFM69W_69HW.DIO4
- removed net R1_DIO5: RFM69W_69HW.DIO5
- removed net R1_LED1: LED4.C
- removed net R1_LED2: LED5.C
- removed net R1_NSS: RFM22B_23B_26W.NSEL, RFM69W_69HW.NSS
- removed net R1_RESET: RFM22B_23B_26W.SDN, RFM69W_69HW.RESET
- removed net R2_DIO1: RFM22B_23B_26W1.GPIO1, RFM69W_69HW1.DIO1
- removed net R2_DIO3: RFM22B_23B_26W1.GPIO3, RFM69W_69HW1.DIO3
- removed net R2_DIO4: RFM22B_23B_26W1.NIRQ, RFM69W_69HW1.DIO4
- removed net R2_DIO5: RFM69W_69HW1.DIO5
- removed net R2_LED1: LED6.C
- removed net R2_LED2: LED7.C
- removed net R2_NSS: RFM22B_23B_26W1.NSEL, RFM69W_69HW1.NSS
- removed net R2_RESET: RFM22B_23B_26W1.SDN, RFM69W_69HW1.RESET
- new net BTN: IC7.PA0, R3.2, R34.1, R35.1, R36.1, R37.1
- new net CODEC_RST: IC7.PB2, IC9.RESET
- new net FLASH1_CS: IC7.PB9, IC8.CS
- new net LCD_CD: IC7.PB1, LCD1.CD
- new net LCD_CS: IC7.PB0, LCD1.CS
- new net N$60: C60.1, LCD1.VB0-
- new net N$61: C61.1, LCD1.VB1-
- new net N$62: C60.2, LCD1.VB0+
- new net N$63: C61.2, LCD1.VB1+
- new net N$64: C62.1, LCD1.VLCD
- new net R12_RESET: IC7.PA10, RFM22B_23B_26W.SDN, RFM22B_23B_26W1.SDN, RFM69W_69HW.RESET, RFM69W_69HW1.RESET
- new net R1_CS: IC7.PA4, RFM22B_23B_26W.NSEL, RFM69W_69HW.NSS
- new net R1_IRQ0: IC7.PC7, RFM22B_23B_26W.NIRQ, RFM69W_69HW.DIO0
- new net R1_IRQ1: IC7.PC8, RFM22B_23B_26W.GPIO1, RFM69W_69HW.DIO1
- new net R1_LED: IC7.PC0, LED4.C
- new net R2_CS: IC7.PA8, RFM22B_23B_26W1.NSEL, RFM69W_69HW1.NSS
- new net R2_IRQ0: IC7.PC4, RFM22B_23B_26W1.NIRQ, RFM69W_69HW1.DIO0
- new net R2_IRQ1: IC7.PC5, RFM22B_23B_26W1.GPIO1, RFM69W_69HW1.DIO1
- new net R2_LED: IC7.PC1, LED5.C
- new net SPI1_MISO: IC7.PA6, IC8.SO, RFM22B_23B_26W.SDO, RFM22B_23B_26W1.SDO, RFM69W_69HW.MISO, RFM69W_69HW1.MISO
- new net SPI1_MOSI: IC7.PA7, IC8.SI, LCD1.SDA, RFM22B_23B_26W.SDI, RFM22B_23B_26W1.SDI, RFM69W_69HW.MOSI, RFM69W_69HW1.MOSI
- new net SPI1_SCK: IC7.PA5, IC8.CLK, LCD1.SCK, RFM22B_23B_26W.SCK, RFM22B_23B_26W1.SCK, RFM69W_69HW.SCK, RFM69W_69HW1.SCK
- net +3V3: now also C59.2, C63.1, IC8.VCC, LCD1.VDD1, LCD1.VDD23; no longer R26.2, R27.2, RFM69W_69HW.VCC, RFM69W_69HW1.VCC
- net BTN1: now also R34.2; no longer IC7.PA3, S1.P
- net BTN2: now also R35.2; no longer IC7.PA2, S2.P
- net BTN3: now also R36.2; no longer IC7.PA1, S3.P
- net BTN4: now also R37.2; no longer IC7.PA0, R3.2, S4.P
- net CHG_CHG: now also IC2.IO0
- net GND: now also C59.1, C62.2, C63.2, C64.2, C65.2, IC8.GND, LCD1.VSS@1, LCD1.VSS@2
- net GPS_LED: now also IC7.PC2
- net GPS_PPS: now also IC7.PB10
- net GPS_PWR: now also IC7.PC3
- net N$56: now also C65.1, RFM69W_69HW1.VCC
- net N$6: now also C64.1, RFM69W_69HW.VCC
- net R1_DIO0: no longer RFM69W_69HW.DIO0
- net R1_DIO2: no longer RFM69W_69HW.DIO2
- net R2_DIO0: no longer RFM69W_69HW1.DIO0
- net R2_DIO2: no longer RFM69W_69HW1.DIO2
- net SCL: now also IC7.PB6
- net SDA: now also IC7.PB7
- net SD_LED: now also IC7.PB5
- net SD_PWR: now also IC7.PB8
- net USART2_RX: now also IC7.PA3
- net USART2_TX: now also IC7.PA2
- net VBAT15_U: now also IC7.PA1
Other:
- note added: "(the S4 button is used for wake-up)"
- note added: "128x64 pixel LCD display"
- note added: "GPS receiver"
- note added: "I2C1"
- note added: "SPI NOR flash memory"
- note added: "SPI1"
- note added: "TODO: check HOLD and WP"
- note added: "TODO: connect CODEC_RESET"
- note added: "TODO: connect I2C"
- note added: "TODO: connect SD_PWR and SD_LED"
- note added: "TODO: power disconnect"
- note removed: "One button needs to be active-high (STM32 wakeup requirement). All buttons are wired the same way to maintain consistency."
- note removed: "TODO: audio codec power disconnect"
- note removed: "TODO: connect either to a SPI port (if at least one is left) or to a GPIO pins. Can be shared with the SPI flash."
- note removed: "TODO: connect to a SPI port. (can be shared with the LCD)"
- moved on the sheet: C1, C44, C45, C46, C47, C56, C57, IC8, LCD1, LED1, LED2, LED4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
